File: hardware/digital_delay/digital_delay.kicad_sch (KiCad schematic)
At the start: 1 part, among them U1 STM32H750XBHx

Commit message: howdy incomplete schematic
Parts:
- added J1: USB_C_Receptacle_USB2.0_16P, symbol Connector:USB_C_Receptacle_USB2.0_16P
- added J2: Conn_01x04, symbol Connector_Generic:Conn_01x04
- added J3: Conn_01x40, Connector_FFC-FPC:Hirose_FH12-40S-0.5SH_1x40-1MP_P0.50mm_Horizontal, symbol Connector_Generic:Conn_01x40
- added U2: PCM3060, Package_SO:TSSOP-28_4.4x9.7mm_P0.65mm, symbol Audio:PCM3060
Connections:
- net +3.3V: now also J3.4 (Pin_4), U2.7 (V_{DD})
- net GND: now also J1.A1 (GND), J1.A12 (GND), J1.B1 (GND), J1.B12 (GND), J1.S1 (SHIELD), J2.2 (Pin_2), J2.4 (Pin_4), J3.29 (Pin_29), J3.3 (Pin_3), J3.36 (Pin_36), U2.16 (SGND), U2.22 (AGND2), U2.23 (AGND1), U2.8 (DGND)
- net LTDC_B0: now also J3.21 (Pin_21)
- net LTDC_B1: now also J3.22 (Pin_22)
- net LTDC_B2: now also J3.23 (Pin_23)
- net LTDC_B3: now also J3.24 (Pin_24)
- net LTDC_CLK: now also J3.30 (Pin_30)
- net LTDC_G0: now also J3.13 (Pin_13)
- net LTDC_G1: now also J3.14 (Pin_14); no longer U1.G15 (PG6)
- net LTDC_G2: now also J3.15 (Pin_15)
- net LTDC_G3: now also J3.16 (Pin_16)
- net LTDC_G4: now also J3.17 (Pin_17)
- net LTDC_G7: now also J3.20 (Pin_20)
- net LTDC_R0: now also J3.5 (Pin_5)
- net LTDC_R1: now also U1.N6 (PJ0), J3.6 (Pin_6); no longer U1.N3 (PA2)
- net LTDC_R2: now also J3.7 (Pin_7)
- net LTDC_R3: now also J3.8 (Pin_8)
- net LTDC_R4: now also J3.9 (Pin_9)
- net LTDC_R5: now also J3.10 (Pin_10)
- net LTDC_R6: now also J3.11 (Pin_11)
- net LTDC_G6: now reaches U1.A15 (PI1)
- net LTDC_G6: now also J3.19 (Pin_19)
- net LTDC_G5: now reaches U1.A16 (PI0)
- net LTDC_G5: now also J3.18 (Pin_18)
- net LTDC_B6: now reaches U1.A2 (PI6)
- net LTDC_B6: now also J3.27 (Pin_27)
- net LTDC_B5: now reaches U1.A3 (PI5)
- net LTDC_B5: now also J3.26 (Pin_26)
- net LTDC_B4: now reaches U1.A4 (PI4)
- net LTDC_B4: now also J3.25 (Pin_25)
- net LTDC_B7: now reaches U1.B3 (PI7)
- net LTDC_B7: now also J3.28 (Pin_28)
- net LTDC_DE: now reaches U1.D7 (PK7)
- net LTDC_DE: now also J3.34 (Pin_34)
- net LTDC_VSYNC: now reaches U1.E2 (PI9)
- net LTDC_VSYNC: now also J3.33 (Pin_33)
- net LTDC_HSYNC: now reaches U1.F3 (PI10)
- net LTDC_HSYNC: now also J3.32 (Pin_32)
- net ADC3_IN5: now reaches U1.H4 (PF3)
- net ADC3_IN4: now reaches U1.J4 (PF5)
- net ADC3_IN9: now reaches U1.J5 (PF4)
- net ADC3_IN8: now reaches U1.K2 (PF6)
- net ADC3_IN3: now reaches U1.K3 (PF7)
- net ADC3_IN7: now reaches U1.K4 (PF8)
- net ADC3_IN10: now reaches U1.L2 (PC0)
- net ADC3_IN6: now reaches U1.L3 (PF10)
- net ADC3_IN2: now reaches U1.L4 (PF9)
- net ADC3_IN11: now reaches U1.M2 (PC1)
- net ADC3_IN12: now reaches U1.M3 (PC2)
- net ADC3_IN13: now reaches U1.N2 (PH2)
- net ADC1_IN17: now reaches U1.N4 (PA1)
- net ADC1_IN16: now reaches U1.N5 (PA0)
- net ADC3_IN14: now reaches U1.P2 (PH3)
- net ADC3_IN15: now reaches U1.P3 (PH4)
- net ADC3_IN16: now reaches U1.P4 (PH5)
- net ADC3_IN0: now reaches U1.R1 (PC2_C)
- net ADC3_IN1: now reaches U1.R2 (PC3_C)
- net ADC1_IN3: now reaches U1.R3 (PA6)
- net ADC1_IN1: now reaches U1.T2 (PA1_C)
- net ADC1_IN19: now reaches U1.T3 (PA5)
- net ADC1_IN15: now reaches U1.U2 (PA3)
- net ADC1_IN18: now reaches U1.U3 (PA4)
- net Disp_EN: now reaches U1.U5 (PB0)
- net Disp_EN: now also J3.31 (Pin_31)
- new net: J2.1 (Pin_1), U2.20 (V_{OUT}L+)
- new net: J2.3 (Pin_3), U2.18 (V_{OUT}R+)
- new net +4.75V: U2.24 (V_{CC})
- new net LEDA: J3.2 (Pin_2)
- new net LEDK: J3.1 (Pin_1)
- new net LTDC_R7: J3.12 (Pin_12), U1.G15 (PG6)
- new net V_in: J1.A4 (VBUS), J1.A9 (VBUS), J1.B4 (VBUS), J1.B9 (VBUS)
- no-connect marks 0 -> 5
Other:
- added sheet Power (Power.kicad_sch)
- moved on the sheet: U1

Commit message: rough design 0.1
Parts:
- added C28, C29, C30, C31: 18p, Capacitor_SMD:C_0201_0603Metric_Pad0.64x0.40mm_HandSolder, symbol Device:C
- added C32: 100n, Capacitor_SMD:C_0201_0603Metric_Pad0.64x0.40mm_HandSolder, symbol Device:C
- added C33: 10u, Capacitor_SMD:C_0201_0603Metric_Pad0.64x0.40mm_HandSolder, symbol Device:C
- added J4: Conn_01x02, Connector_PinHeader_2.54mm:PinHeader_1x02_P2.54mm_Vertical, symbol Connector_Generic:Conn_01x02
- added J5, J6: Conn_02x10_Top_Bottom, Connector_PinHeader_2.54mm:PinHeader_2x10_P2.54mm_Vertical, symbol Connector_Generic:Conn_02x10_Top_Bottom
- added J8: Conn_02x06_Counter_Clockwise, symbol Connector_Generic:Conn_02x06_Counter_Clockwise
- added R1, R2, R4: 220k, Resistor_SMD:R_0201_0603Metric_Pad0.64x0.40mm_HandSolder, symbol Device:R
- added R3: 4k7, Resistor_SMD:R_0201_0603Metric_Pad0.64x0.40mm_HandSolder, symbol Device:R
- added Y1, Y2: Crystal, Crystal:Crystal_SMD_0603-2Pin_6.0x3.5mm, symbol Device:Crystal
- J2: footprint (none) -> Connector_PinHeader_2.54mm:PinHeader_1x04_P2.54mm_Vertical
Connections:
- net +3.3V: now also J8.1 (Pin_1), J8.7 (Pin_7), R1.2, R2.2, R4.2
- net GND: now also U2.27 (~{MS}/AD/IFMD), C28.2, C29.2, C30.2, C31.2, C32.2, C33.2, J4.2 (Pin_2), J8.12 (Pin_12), J8.6 (Pin_6), R3.2
- net V_in: now also J4.1 (Pin_1)
- net Vout_L: now reaches J2.1 (Pin_1), U2.20 (V_{OUT}L+)
- net Vout_R: now reaches J2.3 (Pin_3), U2.18 (V_{OUT}R+)
- net at U2.1 (MC/SCL/FMT): now also R4.1
- net DAC_BCLK: now reaches U2.10 (BCK2)
- net DAC_LRCLK: now reaches U2.11 (LRCK2)
- net DAC_DIN: now reaches U2.12 (DIN)
- net ZERO_F_R: now reaches U2.13 (ZEROR)
- net ZERO_F_L: now reaches U2.14 (ZEROL)
- net at U2.15 (~{RST}): now also R2.1
- net at U2.2 (MD/SDA/DEMP): now also R3.1
- net Vcom: now reaches U2.21 (V_{COM})
- net Vcom: now also C32.1, C33.1
- net Vin_L: now reaches U2.25 (V_{IN}L)
- net Vin_R: now reaches U2.26 (V_{IN}R)
- net at U2.28 (MODE): now also R1.1
- net ADC_DIN: now reaches U2.3 (DOUT)
- net ADC_LRCLK: now reaches U2.4 (LRCK1)
- net ADC_BCLK: now reaches U2.5 (BCK1)
- net ADC_SCLK: now reaches U2.6 (SCKI1)
- net ADC_SCLK: now also U1.C3 (PE2)
- net DAC_SCLK: now reaches U2.9 (SCKI2)
- net USB_DP: now reaches J1.A6 (D+)
- net USB_DP: now also J1.B6 (D+)
- net USB_DM: now reaches J1.A7 (D-)
- net USB_DM: now also J1.B7 (D-)
- net JTAG_DI: now reaches U1.A14 (PA15)
- net JTAG_DI: now also J8.10 (Pin_10), J8.4 (Pin_4)
- net JTAG_CLK: now reaches U1.B14 (PA14)
- net JTAG_CLK: now also J8.3 (Pin_3), J8.9 (Pin_9)
- net OSC32_OUT: now reaches U1.C1 (PC15)
- net OSC32_OUT: now also C30.1, Y1.1
- net JTAG_MS: now reaches U1.C15 (PA13)
- net JTAG_MS: now also J8.2 (Pin_2), J8.8 (Pin_8)
- net OSC32_IN: now reaches U1.C2 (PC14)
- net OSC32_IN: now also C28.1, Y1.2
- net JTAG_DO: now reaches U1.C6 (PB3)
- net JTAG_DO: now also J8.11 (Pin_11), J8.5 (Pin_5)
- net I2S_CLK_IN: now reaches U1.E14 (PC9)
- net OSC_OUT: now reaches U1.J1 (PH1)
- net OSC_OUT: now also C31.1, Y2.1
- net OSC_IN: now reaches U1.J2 (PH0)
- net OSC_IN: now also C29.1, Y2.2
- no-connect marks 5 -> 7
Other:
- moved on the sheet: J1, J2, J3, U1, U2
