File: hardware/digital_delay/digital_delay.kicad_sch (KiCad schematic)
At the start: 21 parts, among them J1 USB_C_Receptacle_USB2.0_16P, J2 Conn_01x04, J3 Conn_01x40, J4 Conn_01x02, J5 Conn_02x10_Top_Bottom, J6 Conn_02x10_Top_Bottom, J8 Conn_02x06_Counter_Clockwise, U1 STM32H750XBHx, U2 PCM3060, Y1 Crystal, Y2 Crystal

Commit message: memory
Parts:
- added U6: MT48LC16M16A2P, Package_SO:TSOP-II-54_22.2x10.16mm_P0.8mm, symbol Memory_RAM:MT48LC16M16A2P
Connections:
- net +3.3V: now also U6.1 (VDD), U6.14 (VDD), U6.27 (VDD), U6.3 (VDDQ), U6.43 (VDDQ), U6.49 (VDDQ), U6.9 (VDDQ)
- net GND: now also U6.12 (VSSQ), U6.28 (VSS), U6.41 (VSS), U6.46 (VSSQ), U6.52 (VSSQ), U6.54 (VSS), U6.6 (VSSQ)
- new net FMC_A0: U6.23 (A0)
- new net FMC_A1: U6.24 (A1)
- new net FMC_A10: U6.22 (A10)
- new net FMC_A11: U6.35 (A11)
- new net FMC_A12: U6.36 (A12)
- new net FMC_A2: U6.25 (A2)
- new net FMC_A3: U6.26 (A3)
- new net FMC_A4: U6.29 (A4)
- new net FMC_A5: U6.30 (A5)
- new net FMC_A6: U6.31 (A6)
- new net FMC_A7: U6.32 (A7)
- new net FMC_A8: U6.33 (A8)
- new net FMC_A9: U6.34 (A9)
- new net FMC_B0: U6.20 (BA0)
- new net FMC_B1: U6.21 (BA1)
- new net FMC_CAS: U6.17 (~{CAS})
- new net FMC_CKE: U6.37 (CKE)
- new net FMC_CLK: U6.38 (CLK)
- new net FMC_CS: U6.19 (~{CS})
- new net FMC_D0: U6.2 (DQ0)
- new net FMC_D1: U6.4 (DQ1)
- new net FMC_D10: U6.45 (DQ10)
- new net FMC_D11: U6.47 (DQ11)
- new net FMC_D12: U6.48 (DQ12)
- new net FMC_D13: U6.50 (DQ13)
- new net FMC_D14: U6.51 (DQ14)
- new net FMC_D15: U6.53 (DQ15)
- new net FMC_D2: U6.5 (DQ2)
- new net FMC_D3: U6.7 (DQ3)
- new net FMC_D4: U6.8 (DQ4)
- new net FMC_D5: U6.10 (DQ5)
- new net FMC_D6: U6.11 (DQ6)
- new net FMC_D7: U6.13 (DQ7)
- new net FMC_D8: U6.42 (DQ8)
- new net FMC_D9: U6.44 (DQ9)
- new net FMC_DQMH: U6.39 (DQMH)
- new net FMC_DQML: U6.15 (DQML)
- new net FMC_RAS: U6.18 (~{RAS})
- new net FMC_WE: U6.16 (~{WE})
